File: sample_holder.sch (KiCad schematic (older format))
At the start: 14 parts, among them J1 Conn_Coaxial, J10 RF_Shield_One_Piece, J2 Conn_Coaxial, J3 Conn_Coaxial, J4 Conn_Coaxial, J5 Conn_Coaxial, J6 Conn_Coaxial, J7 Conn_Coaxial, J8 Conn_Coaxial, U1 sample

Commit message: fix up libraries
Parts:
- J1, J2, J3, J4, J5, J6, J7, J8: footprint imp:0732513481 -> sample_holder:0732513481
Changed lines of the file:
@@
 F 0 "J8" H 4450 3400 50  0000 L CNN
 F 1 "Conn_Coaxial" H 4450 3373 50  0001 L CNN
-F 2 "imp:0732513481" H 4350 3400 50  0001 C CNN
+F 2 "sample_holder:0732513481" H 4350 3400 50  0001 C CNN
 F 3 " ~" H 4350 3400 50  0001 C CNN
 	1    4350 3400
@@
 F 0 "J7" H 4450 3800 50  0000 L CNN
 F 1 "Conn_Coaxial" H 4450 3773 50  0001 L CNN
-F 2 "imp:0732513481" H 4350 3800 50  0001 C CNN
+F 2 "sample_holder:0732513481" H 4350 3800 50  0001 C CNN
 F 3 " ~" H 4350 3800 50  0001 C CNN
 	1    4350 3800
@@
 F 0 "J1" V 5300 2600 50  0000 C CNN
 F 1 "Conn_Coaxial" V 5296 2529 50  0001 C CNN
-F 2 "imp:0732513481" H 5150 2600 50  0001 C CNN
+F 2 "sample_holder:0732513481" H 5150 2600 50  0001 C CNN
 F 3 " ~" H 5150 2600 50  0001 C CNN
 	1    5150 2600
@@
 F 0 "J3" H 6450 3400 50  0000 L CNN
 F 1 "Conn_Coaxial" H 6450 3284 50  0001 L CNN
-F 2 "imp:0732513481" H 6350 3400 50  0001 C CNN
+F 2 "sample_holder:0732513481" H 6350 3400 50  0001 C CNN
 F 3 " ~" H 6350 3400 50  0001 C CNN
 	1    6350 3400
@@
 F 0 "J4" H 6450 3800 50  0000 L CNN
 F 1 "Conn_Coaxial" H 6450 3684 50  0001 L CNN
-F 2 "imp:0732513481" H 6350 3800 50  0001 C CNN
+F 2 "sample_holder:0732513481" H 6350 3800 50  0001 C CNN
 F 3 " ~" H 6350 3800 50  0001 C CNN
 	1    6350 3800
@@
 F 0 "J5" V 5600 4700 50  0000 L CNN
 F 1 "Conn_Coaxial" V 5573 4700 50  0001 L CNN
-F 2 "imp:0732513481" H 5600 4600 50  0001 C CNN
+F 2 "sample_holder:0732513481" H 5600 4600 50  0001 C CNN
 F 3 " ~" H 5600 4600 50  0001 C CNN
 	1    5600 4600
@@
 F 0 "J6" V 5100 4700 50  0000 L CNN
 F 1 "Conn_Coaxial" V 5073 4700 50  0001 L CNN
-F 2 "imp:0732513481" H 5100 4600 50  0001 C CNN
+F 2 "sample_holder:0732513481" H 5100 4600 50  0001 C CNN
 F 3 " ~" H 5100 4600 50  0001 C CNN
 	1    5100 4600
@@
 F 0 "J2" V 5700 2600 50  0000 C CNN
 F 1 "Conn_Coaxial" V 5696 2529 50  0001 C CNN
-F 2 "imp:0732513481" H 5550 2600 50  0001 C CNN
+F 2 "sample_holder:0732513481" H 5550 2600 50  0001 C CNN
 F 3 " ~" H 5550 2600 50  0001 C CNN
 	1    5550 2600
